File: ACNode.brd (EAGLE design)
At the start: 100 x 65 mm, 97 parts, among them IC1 74AHC1G04DCK, IC2 MC78M05CDTG, IC3 LM1117IMP-3.3, IC4 MC78M05CDTG, IC5 ULN2003AN, J1 POWER_JACKPTH, K1 351, T1 MMBT4401, U2 MAGJACK-POE, U3 CLAMP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

Commit message: Correct DRC
Routing:
- net N$16: track 50.2 -> 45.7 mm
- net N$32: track 15.8 -> 13.4 mm
- net +3V3: track 71.0 -> 68.7 mm
- net GND: track 52.1 -> 52.9 mm
- net RAW: track 228.3 -> 229.0 mm
Changed lines of the file:
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@@
 necessary adjustments and save your customized
 design rules under a new name.</description>
+<description language="zh">&lt;b&gt;Seeed Studio EAGLE Design Rules&lt;/b&gt;
+</description>
 <param name="layerSetup" value="(1*16)"/>
 <param name="mtCopper" value="0.035mm 0.035mm 0.035mm 0.035mm 0.035mm 0.035mm 0.035mm 0.035mm 0.035mm 0.035mm 0.035mm 0.035mm 0.035mm 0.035mm 0.035mm 0.035mm"/>
 <param name="mtIsolate" value="1.5mm 0.15mm 0.2mm 0.15mm 0.2mm 0.15mm 0.2mm 0.15mm 0.2mm 0.15mm 0.2mm 0.15mm 0.2mm 0.15mm 0.2mm"/>
-<param name="mdWireWire" value="8mil"/>
-<param name="mdWirePad" value="8mil"/>
-<param name="mdWireVia" value="8mil"/>
-<param name="mdPadPad" value="8mil"/>
-<param name="mdPadVia" value="8mil"/>
-<param name="mdViaVia" value="8mil"/>
-<param name="mdSmdPad" value="8mil"/>
-<param name="mdSmdVia" value="8mil"/>
-<param name="mdSmdSmd" value="8mil"/>
+<param name="mdWireWire" value="6mil"/>
+<param name="mdWirePad" value="6mil"/>
+<param name="mdWireVia" value="6mil"/>
+<param name="mdPadPad" value="6mil"/>
+<param name="mdPadVia" value="6mil"/>
+<param name="mdViaVia" value="6mil"/>
+<param name="mdSmdPad" value="0mil"/>
+<param name="mdSmdVia" value="0mil"/>
+<param name="mdSmdSmd" value="0mil"/>
 <param name="mdViaViaSameLayer" value="8mil"/>
 <param name="mnLayersViaInSmd" value="2"/>
-<param name="mdCopperDimension" value="40mil"/>
-<param name="mdDrill" value="8mil"/>
+<param name="mdCopperDimension" value="10mil"/>
+<param name="mdDrill" value="10mil"/>
 <param name="mdSmdStop" value="0mil"/>
-<param name="msWidth" value="10mil"/>
-<param name="msDrill" value="24mil"/>
-<param name="msMicroVia" value="9.99mm"/>
+<param name="msWidth" value="6mil"/>
+<param name="msDrill" value="12mil"/>
+<param name="msMicroVia" value="12mil"/>
 <param name="msBlindViaRatio" value="0.5"/>
 <param name="rvPadTop" value="0.25"/>
@@
 <param name="rlMinPadBottom" value="10mil"/>
 <param name="rlMaxPadBottom" value="20mil"/>
-<param name="rlMinViaOuter" value="8mil"/>
+<param name="rlMinViaOuter" value="6mil"/>
 <param name="rlMaxViaOuter" value="20mil"/>
-<param name="rlMinViaInner" value="8mil"/>
+<param name="rlMinViaInner" value="6mil"/>
 <param name="rlMaxViaInner" value="20mil"/>
 <param name="rlMinMicroViaOuter" value="4mil"/>
@@
 <param name="psTop" value="-1"/>
 <param name="psBottom" value="-1"/>
-<param name="psFirst" value="-1"/>
+<param name="psFirst" value="0"/>
 <param name="psElongationLong" value="100"/>
 <param name="psElongationOffset" value="100"/>
 <param name="mvStopFrame" value="1"/>
 <param name="mvCreamFrame" value="0"/>
-<param name="mlMinStopFrame" value="4mil"/>
-<param name="mlMaxStopFrame" value="4mil"/>
+<param name="mlMinStopFrame" value="2mil"/>
+<param name="mlMaxStopFrame" value="2mil"/>
 <param name="mlMinCreamFrame" value="0mil"/>
 <param name="mlMaxCreamFrame" value="0mil"/>
-<param name="mlViaStopLimit" value="0mil"/>
+<param name="mlViaStopLimit" value="100mil"/>
 <param name="srRoundness" value="0"/>
 <param name="srMinRoundness" value="0mil"/>
@@
 <param name="checkAngle" value="0"/>
 <param name="checkFont" value="1"/>
-<param name="checkRestrict" value="1"/>
+<param name="checkRestrict" value="0"/>
 <param name="useDiameter" value="13"/>
 <param name="maxErrors" value="50"/>
@@
 <wire x1="25.85" y1="26.4" x2="25.85" y2="26.2" width="0.4064" layer="1"/>
 <wire x1="25.85" y1="26.2" x2="24.6" y2="26.2" width="0.4064" layer="1"/>
-<wire x1="27.8" y1="36.55" x2="28.2" y2="36.55" width="0.4064" layer="1"/>
 <wire x1="29" y1="36.55" x2="29" y2="37.8" width="0.2" layer="1"/>
 <wire x1="30.2" y1="36.55" x2="30.2" y2="37.8" width="0.2" layer="1"/>
@@
 <wire x1="23.2" y1="22.4" x2="23.4" y2="22.2" width="0.8128" layer="1"/>
 <contactref element="J1" pad="PWR"/>
+<wire x1="28.2" y1="36.55" x2="28.2" y2="37.8" width="0.2" layer="1"/>
 </signal>
 <signal name="N$6">
@@
 <wire x1="29.4" y1="23.2" x2="30.2" y2="23.2" width="0.2" layer="1"/>
 <via x="21" y="27.6" extent="1-16" drill="0.6" shape="square"/>
-<wire x1="21" y1="27.6" x2="22.8" y2="26.2" width="0.6096" layer="16"/>
 <wire x1="28.6" y1="36.55" x2="28.6" y2="35" width="0.2" layer="1"/>
 <via x="28.6" y="35" extent="1-16" drill="0.6" shape="square"/>
@@
 <contactref element="U1" pad="70"/>
 <contactref element="U2" pad="12"/>
-<wire x1="1.92" y1="40.085" x2="8.4" y2="33.605" width="0.2" layer="1"/>
-<wire x1="8.4" y1="33.605" x2="8.4" y2="29.8" width="0.2" layer="1"/>
-<wire x1="8.4" y1="29.8" x2="7.2" y2="28.6" width="0.2" layer="1"/>
-<wire x1="7.2" y1="28.6" x2="7.2" y2="27.6" width="0.2" layer="1"/>
-<wire x1="7.2" y1="27.6" x2="10.4" y2="24.4" width="0.2" layer="1"/>
-<wire x1="10.4" y1="24.4" x2="25.6" y2="24.4" width="0.2" layer="1"/>
+<wire x1="1.92" y1="40.085" x2="11.2" y2="30.805" width="0.2" layer="1"/>
 <wire x1="25.6" y1="24.4" x2="26.4" y2="25.2" width="0.2" layer="1"/>
 <wire x1="26.4" y1="25.2" x2="26.4" y2="26" width="0.2" layer="1"/>
@@
 <wire x1="27.4" y1="27" x2="32.4" y2="27" width="0.2" layer="1"/>
 <wire x1="32.4" y1="27" x2="36" y2="30.6" width="0.2" layer="1"/>
+<wire x1="12.4" y1="28.4" x2="13.8" y2="28.4" width="0.2" layer="1"/>
+<wire x1="13.8" y1="28.4" x2="17.8" y2="24.4" width="0.2" layer="1"/>
+<wire x1="17.8" y1="24.4" x2="25.6" y2="24.4" width="0.2" layer="1"/>
+<wire x1="11.2" y1="30.805" x2="11.2" y2="29.6" width="0.2" layer="1"/>
+<wire x1="11.2" y1="29.6" x2="12.4" y2="28.4" width="0.2" layer="1"/>
 </signal>
 <signal name="N$17">
@@
 <wire x1="35" y1="29.8" x2="41" y2="29.8" width="0.2" layer="16"/>
 <wire x1="41" y1="29.8" x2="42.6" y2="31.4" width="0.2" layer="16"/>
-<wire x1="42.6" y1="31.4" x2="63.2" y2="31.4" width="0.2" layer="16"/>
-<wire x1="63.2" y1="31.4" x2="64.2" y2="32.4" width="0.2" layer="16"/>
-<wire x1="64.2" y1="32.4" x2="68" y2="32.4" width="0.2" layer="16"/>
+<wire x1="42.6" y1="31.4" x2="63.8" y2="31.4" width="0.2" layer="16"/>
+<wire x1="63.8" y1="31.4" x2="64.8" y2="32.4" width="0.2" layer="16"/>
+<wire x1="64.8" y1="32.4" x2="68" y2="32.4" width="0.2" layer="16"/>
 <via x="69.2" y="32" extent="1-16" drill="0.6" shape="square"/>
 <wire x1="68" y1="32.4" x2="68.4" y2="32" width="0.2" layer="16"/>
@@
 <wire x1="35.2" y1="30.2" x2="40.8" y2="30.2" width="0.2" layer="16"/>
 <wire x1="40.8" y1="30.2" x2="42.4" y2="31.8" width="0.2" layer="16"/>
-<wire x1="42.4" y1="31.8" x2="62.8" y2="31.8" width="0.2" layer="16"/>
-<wire x1="62.8" y1="31.8" x2="64.2" y2="33.2" width="0.2" layer="16"/>
-<wire x1="64.2" y1="33.2" x2="69.2" y2="33.2" width="0.2" layer="16"/>
+<wire x1="42.4" y1="31.8" x2="63.4" y2="31.8" width="0.2" layer="16"/>
+<wire x1="63.4" y1="31.8" x2="64.8" y2="33.2" width="0.2" layer="16"/>
+<wire x1="64.8" y1="33.2" x2="69.2" y2="33.2" width="0.2" layer="16"/>
 <via x="69.2" y="33.2" extent="1-16" drill="0.6" shape="square"/>
 <wire x1="69.2" y1="33.2" x2="66.4926" y2="33.2" width="0.2" layer="1"/>
@@
 <wire x1="28.6" y1="33.6" x2="33.6" y2="33.6" width="0.2" layer="16"/>
 <wire x1="33.6" y1="33.6" x2="35" y2="32.2" width="0.2" layer="16"/>
-<wire x1="35" y1="32.2" x2="62.4" y2="32.2" width="0.2" layer="16"/>
-<wire x1="62.4" y1="32.2" x2="64.2" y2="34" width="0.2" layer="16"/>
+<wire x1="35" y1="32.2" x2="63" y2="32.2" width="0.2" layer="16"/>
+<wire x1="63" y1="32.2" x2="64.8" y2="34" width="0.2" layer="16"/>
 <via x="69.2" y="34.4" extent="1-16" drill="0.6" shape="square"/>
-<wire x1="64.2" y1="34" x2="67.4" y2="34" width="0.2" layer="16"/>
+<wire x1="64.8" y1="34" x2="67.4" y2="34" width="0.2" layer="16"/>
 <wire x1="67.4" y1="34" x2="67.8" y2="34.4" width="0.2" layer="16"/>
 <wire x1="67.8" y1="34.4" x2="69.2" y2="34.4" width="0.2" layer="16"/>
@@
 <wire x1="52.4" y1="6.6" x2="54" y2="5" width="0.8128" layer="16"/>
 <wire x1="54" y1="5" x2="54" y2="2.4" width="0.8128" layer="16"/>
-<wire x1="54" y1="2.4" x2="55" y2="1.4" width="0.8128" layer="16"/>
-<wire x1="55" y1="1.4" x2="97.2" y2="1.4" width="0.8128" layer="16"/>
-<wire x1="97.2" y1="1.4" x2="97.6" y2="1.8" width="0.8128" layer="16"/>
+<wire x1="54" y1="2.4" x2="55.8" y2="0.6" width="0.8128" layer="16"/>
 <wire x1="97.6" y1="1.8" x2="97.6" y2="6.6" width="0.8128" layer="16"/>
 <wire x1="97.6" y1="6.6" x2="96.4" y2="7.8" width="0.8128" layer="16"/>
@@
 <wire x1="6.4" y1="20" x2="3" y2="16.6" width="0.8128" layer="16"/>
 <wire x1="3" y1="16.6" x2="3.1" y2="16.6" width="0.8128" layer="16"/>
+<wire x1="97.6" y1="1.8" x2="96.4" y2="0.6" width="0.8128" layer="16"/>
+<wire x1="96.4" y1="0.6" x2="55.8" y2="0.6" width="0.8128" layer="16"/>
 </signal>
 <signal name="N$26">
@@
 <contactref element="K1" pad="S1"/>
 <contactref element="RELAY" pad="6"/>
-<wire x1="87.41" y1="51.77" x2="94.77" y2="51.77" width="0.8128" layer="1"/>
-<wire x1="94.77" y1="51.77" x2="96.8" y2="53.8" width="0.8128" layer="1"/>
-<wire x1="96.8" y1="53.8" x2="96.8" y2="58.43" width="0.8128" layer="1"/>
-<wire x1="96.8" y1="58.43" x2="96.7" y2="59.33" width="0.8128" layer="1"/>
+<wire x1="87.41" y1="51.77" x2="90.77" y2="51.77" width="0.8128" layer="1"/>
+<wire x1="90.77" y1="51.77" x2="96.6" y2="57.6" width="0.8128" layer="1"/>
+<wire x1="96.6" y1="57.6" x2="96.6" y2="59.23" width="0.8128" layer="1"/>
+<wire x1="96.6" y1="59.23" x2="96.7" y2="59.33" width="0.8128" layer="1"/>
 </signal>
 <signal name="N$33">
@@
 </signal>
 </signals>
+<errors>
+</errors>
 </board>
 </drawing>

Commit message: Correct SL030 pins
Parts:
- added SJ14: (no value), SparkFun-Passives:SJ_2S-TRACE
- moved C7 1.60 mm to (47.2, 42.8)
- moved SJ3 0.40 mm to (53.4, 10.8)
Connections:
- removed net RFOUT: SL030.5
- new net N$57: SJ14.2, SL030.5
- net +3V3: now also U$2.3, U$2.8
- net A0: now also SJ14.1
- net VCC: no longer U$2.8
Routing:
- net +3V3: track 68.7 -> 96.4 mm
- net VCC: track 80.0 -> 76.9 mm
- net N$20: track 20.0 -> 20.7 mm
Changed lines of the file:
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@@
 <element name="R11" library="SparkFun-Passives" package="0603-RES" value="1M" x="40.8" y="34.6"/>
 <element name="C6" library="SparkFun-Passives" package="0603-CAP" value="18p" x="40.8" y="42.8" rot="R180"/>
-<element name="C7" library="SparkFun-Passives" package="0603-CAP" value="18p" x="48.8" y="42.8"/>
+<element name="C7" library="SparkFun-Passives" package="0603-CAP" value="18p" x="47.2" y="42.8"/>
 <element name="C8" library="SparkFun-Passives" package="0603-CAP" value="0.1uF" x="32.8" y="38.8" rot="R180"/>
 <element name="C9" library="SparkFun-Passives" package="EIA3216" value="1uf / 16v" x="31.8" y="43.8"/>
@@
 <element name="R15" library="SparkFun-Passives" package="0603-RES" value="100" x="23.2" y="12.3"/>
 <element name="LED1" library="SparkFun-LED" package="LED-0603" value="" x="20.2" y="12.3" rot="R90"/>
-<element name="POWER" library="con-wago-500" package="W237-6" value="" x="23.06" y="6.05">
+<element name="POWER" library="con-wago-500" package="W237-6" value="" x="23.06" y="6.05" smashed="yes">
 <attribute name="OC_NEWARK" value="unknown" x="51" y="-38.4" size="1.778" layer="27" display="off"/>
 <attribute name="MPN" value="" x="51" y="-38.4" size="1.778" layer="27" display="off"/>
 <attribute name="MF" value="" x="51" y="-38.4" size="1.778" layer="27" display="off"/>
 <attribute name="OC_FARNELL" value="unknown" x="51" y="-38.4" size="1.778" layer="27" display="off"/>
+<attribute name="VALUE" x="10.4076" y="1.0208" size="1.27" layer="27" ratio="10"/>
+<attribute name="NAME" x="11.017" y="10.3062" size="1.27" layer="25" ratio="10"/>
 </element>
 <element name="IC3" library="SparkFun-PowerIC" package="SOT223" value="LM1117IMP-3.3" x="5.8" y="53.7" rot="R90"/>
@@
 <element name="R16" library="SparkFun-Passives" package="0603-RES" value="100" x="13.2" y="48.8" rot="R90"/>
 <element name="LED2" library="SparkFun-LED" package="LED-0603" value="" x="15" y="48.8"/>
-<element name="INPUT" library="con-wago-500" package="W237-6" value="" x="72.59" y="6.08">
+<element name="INPUT" library="con-wago-500" package="W237-6" value="" x="72.59" y="6.08" smashed="yes">
 <attribute name="OC_NEWARK" value="unknown" x="127.2" y="-24.4" size="1.778" layer="27" display="off"/>
 <attribute name="MPN" value="" x="127.2" y="-24.4" size="1.778" layer="27" display="off"/>
 <attribute name="MF" value="" x="127.2" y="-24.4" size="1.778" layer="27" display="off"/>
 <attribute name="OC_FARNELL" value="unknown" x="127.2" y="-24.4" size="1.778" layer="27" display="off"/>
+<attribute name="VALUE" x="59.9376" y="1.0508" size="1.27" layer="27" ratio="10"/>
+<attribute name="NAME" x="59.147" y="10.5362" size="1.27" layer="25" ratio="10"/>
 </element>
 <element name="K1" library="relay" package="351" value="351" x="83.6" y="37.8" rot="R90">
@@
 <element name="R22" library="SparkFun-Passives" package="0603-RES" value="" x="53.8" y="3.6"/>
 <element name="U3" library="SparkFun-Connectors" package="AUDIO-JACK" value="CLAMP" x="45.4" y="4" rot="R90"/>
-<element name="SJ3" library="SparkFun-Passives" package="SJ_2S-NO" value="SOLDERJUMPERNO" x="53" y="10.8" rot="R90"/>
+<element name="SJ3" library="SparkFun-Passives" package="SJ_2S-NO" value="SOLDERJUMPERNO" x="53.4" y="10.8" rot="R90"/>
 <element name="IC5" library="uln-udn" package="DIL16" value="ULN2003AN" x="83.2" y="20.6" rot="R270"/>
 <element name="X1" library="con-wago-500" package="W237-4" value="" x="95.15" y="40.34" rot="R270">
@@
 <element name="H4" library="holes" package="3,0" value="MOUNT-HOLE3.0" x="4" y="4"/>
 <element name="J1" library="SparkFun-Connectors" package="POWER_JACK_PTH" value="POWER_JACKPTH" x="-4.6" y="16.6" rot="R270"/>
+<element name="SJ14" library="SparkFun-Passives" package="SJ_2S-TRACE" value="" x="-7.2" y="-0.4"/>
 </elements>
 <signals>
@@
 <via x="10.8" y="22.6" extent="1-16" drill="0.6" shape="square"/>
 <wire x1="10.8" y1="22.6" x2="16.2" y2="22.6" width="0.8128" layer="1"/>
+<contactref element="U$2" pad="8"/>
+<wire x1="58.4862" y1="44.725" x2="58.5612" y2="44.8" width="0.3048" layer="1"/>
+<contactref element="U$2" pad="3"/>
+<wire x1="58.4862" y1="44.725" x2="56.925" y2="44.725" width="0.6096" layer="1"/>
+<wire x1="56.925" y1="44.725" x2="55.8" y2="43.6" width="0.6096" layer="1"/>
+<wire x1="55.8" y1="43.6" x2="55.8" y2="43.4" width="0.6096" layer="1"/>
+<wire x1="55.8" y1="43.4" x2="54.6" y2="42.2" width="0.6096" layer="1"/>
+<wire x1="54.6" y1="42.2" x2="53.2688" y2="42.2" width="0.6096" layer="1"/>
+<wire x1="53.2688" y1="42.2" x2="53.2538" y2="42.185" width="0.6096" layer="1"/>
+<wire x1="53.2688" y1="42.2" x2="51.8" y2="42.2" width="0.6096" layer="1"/>
+<wire x1="51.8" y1="42.2" x2="51.2" y2="42.8" width="0.6096" layer="1"/>
+<wire x1="51.2" y1="42.8" x2="51.2" y2="45.6" width="0.6096" layer="1"/>
+<wire x1="51.2" y1="45.6" x2="49" y2="47.8" width="0.6096" layer="1"/>
+<wire x1="49" y1="47.8" x2="36.09" y2="47.8" width="0.6096" layer="1"/>
+<wire x1="36.09" y1="47.8" x2="36.05" y2="47.84" width="0.6096" layer="1"/>
 </signal>
 <signal name="N$9">
@@
 <contactref element="C7" pad="2"/>
 <wire x1="49.626" y1="38.76" x2="49.65" y2="38.784" width="0.4064" layer="1"/>
-<wire x1="49.65" y1="38.784" x2="49.65" y2="42.8" width="0.4064" layer="1"/>
 <wire x1="41.65" y1="34.6" x2="41.65" y2="35.65" width="0.4064" layer="1"/>
 <wire x1="41.65" y1="35.65" x2="42.8" y2="36.8" width="0.4064" layer="1"/>
@@
 <wire x1="41.6" y1="33.6" x2="41.6" y2="34.55" width="0.2" layer="1"/>
 <wire x1="41.6" y1="34.55" x2="41.65" y2="34.6" width="0.2" layer="1"/>
+<wire x1="48.05" y1="42.8" x2="48.05" y2="40.336" width="0.4064" layer="1"/>
+<wire x1="48.05" y1="40.336" x2="49.626" y2="38.76" width="0.4064" layer="1"/>
 </signal>
 <signal name="N$21">
@@
 <contactref element="U$1" pad="6"/>
 <contactref element="R12" pad="2"/>
-<contactref element="U$2" pad="8"/>
 <contactref element="R13" pad="2"/>
 <contactref element="FDTI" pad="4"/>
@@
 <via x="59.6" y="37.8" extent="1-16" drill="0.6" shape="square"/>
 <wire x1="59.6" y1="37.8" x2="59.6" y2="38" width="0.3048" layer="16"/>
-<wire x1="58.4862" y1="44.725" x2="58.5612" y2="44.8" width="0.3048" layer="1"/>
-<wire x1="58.5612" y1="44.8" x2="61.2" y2="44.8" width="0.3048" layer="1"/>
-<via x="61.2" y="44.8" extent="1-16" drill="0.6" shape="square"/>
-<wire x1="61.2" y1="44.8" x2="61.4" y2="44.8" width="0.3048" layer="16"/>
 <wire x1="58.6" y1="32.8" x2="60.2" y2="32.8" width="0.3048" layer="16"/>
 <wire x1="60.2" y1="32.8" x2="61.2" y2="33.8" width="0.3048" layer="16"/>
@@
 <via x="85" y="38.2" extent="1-16" drill="0.6" shape="square"/>
 <wire x1="80.4" y1="38.2" x2="85" y2="38.2" width="0.3048" layer="1"/>
-<via x="58.2" y="46.2" extent="1-16" drill="0.6" shape="square"/>
-<wire x1="58.2" y1="46.2" x2="60.8" y2="46.2" width="0.8128" layer="1"/>
-<wire x1="60.8" y1="46.2" x2="61.2" y2="45.8" width="0.8128" layer="1"/>
-<wire x1="61.2" y1="45.8" x2="61.2" y2="44.8" width="0.8128" layer="1"/>
 <wire x1="61.8" y1="26.9074" x2="61.8" y2="25.6" width="0.4064" layer="1"/>
 <wire x1="61.8" y1="25.6" x2="62.2" y2="25.2" width="0.4064" layer="1"/>
@@
 <wire x1="63" y1="25.2" x2="63.4" y2="25.6" width="0.4064" layer="1"/>
 <wire x1="63.4" y1="25.6" x2="63.4" y2="26.9074" width="0.4064" layer="1"/>
+<wire x1="58.8" y1="47.8" x2="59.8" y2="46.8" width="0.8128" layer="1"/>
+<via x="61.2" y="46.8" extent="1-16" drill="0.6" shape="square"/>
+<wire x1="59.8" y1="46.8" x2="61.2" y2="46.8" width="0.8128" layer="1"/>
+<wire x1="58.8" y1="47.8" x2="57.6" y2="47.8" width="0.8128" layer="1"/>
+<via x="57.6" y="47.8" extent="1-16" drill="0.6" shape="square"/>
 </signal>
 <signal name="RESET">
@@
 <signal name="RFIN">
 <contactref element="SL030" pad="2"/>
-</signal>
-<signal name="RFOUT">
-<contactref element="SL030" pad="5"/>
 </signal>
 <signal name="RAW">
@@
 <contactref element="U$1" pad="26"/>
 <contactref element="SJ3" pad="2"/>
-<wire x1="53" y1="11.25" x2="53" y2="15.4" width="0.4064" layer="1"/>
-<wire x1="53" y1="15.4" x2="52.6" y2="15.8" width="0.4064" layer="1"/>
 <wire x1="52.6" y1="15.8" x2="52.6" y2="21.8" width="0.4064" layer="1"/>
 <wire x1="52.6" y1="21.8" x2="55.6" y2="24.8" width="0.4064" layer="1"/>
@@
 <wire x1="59.4" y1="32.6" x2="58.8" y2="33.2" width="0.4064" layer="1"/>
 <wire x1="58.8" y1="33.2" x2="57.9074" y2="33.2" width="0.4064" layer="1"/>
+<wire x1="52.6" y1="15.8" x2="53.4" y2="15" width="0.4064" layer="1"/>
+<wire x1="53.4" y1="15" x2="53.4" y2="11.25" width="0.4064" layer="1"/>
 </signal>
 <signal name="A2">
@@
 <wire x1="73.6" y1="30.4" x2="75" y2="29" width="0.3048" layer="1"/>
 <wire x1="75" y1="29" x2="75.95" y2="29" width="0.3048" layer="1"/>
+<contactref element="SJ14" pad="1"/>
+<wire x1="-7.708" y1="-0.4" x2="60.2" y2="34.8" width="0" layer="19" extent="1-1"/>
 </signal>
 <signal name="N$40">
@@
 <wire x1="52.95" y1="8.8" x2="50.6" y2="8.8" width="0.6096" layer="1"/>
 <wire x1="50.6" y1="8.8" x2="50.4" y2="9" width="0.6096" layer="1"/>
-<wire x1="53" y1="10.35" x2="53" y2="8.85" width="0.6096" layer="1"/>
 <wire x1="53" y1="8.85" x2="52.95" y2="8.8" width="0.6096" layer="1"/>
+<wire x1="53.4" y1="10.35" x2="52.95" y2="9.9" width="0.4064" layer="1"/>
+<wire x1="52.95" y1="9.9" x2="52.95" y2="8.8" width="0.4064" layer="1"/>
 </signal>
 <signal name="N$42">
@@
 <wire x1="68.8" y1="47.95" x2="68.95" y2="47.8" width="0.4064" layer="1"/>
 </signal>
+<signal name="N$57">
+<contactref element="SL030" pad="5"/>
+<contactref element="SJ14" pad="2"/>
+<wire x1="-6.692" y1="-0.4" x2="25.89" y2="47.84" width="0" layer="19" extent="1-1"/>
+</signal>
 </signals>
-<errors>
-</errors>
 </board>
 </drawing>
