File: ACNode0_3.sch (EAGLE design)
At the start: 85 parts, among them IC1 74AHC1G04DCK, IC2 MC78M05CDTG, IC3 LM1117IMP-3.3, J1 POWER_JACKPTH, K1 351, K2 351, T1 MMBT4401, T2 MMBT4401, U2 MAGJACK-POE, U3 CLAMP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

Commit message: layout sans poe
Parts:
- removed CASE, CASE1: (no value), con-wago-500:W237-4
- removed RELAY: (no value), con-wago-500:W237-6
- added 5V_SSR_CON: (no value), con-wago-500:W237-4
- added RELAY2: (no value), con-wago-500:W237-6
- added X1: (no value), con-wago-500:W237-102
Connections:
- removed net N$44: K23.P, RELAY1-3.KL
- removed net N$45: K22.P, RELAY1-4.KL
- new net N$23: K22.P, RELAY2-3.KL
- new net N$36: K23.P, RELAY2-6.KL
- net +3V3: now also POWER-4.KL, R13.2, R14.2; no longer POWER-2.KL
- net A1: now also JP1.9; no longer JP1.3
- net A2: now also JP1.5; no longer JP1.2
- net A3: now also JP1.7; no longer JP1.1
- net A6: now also SG1.2; no longer CASE1-1.KL, SJ1.2
- net A7: now also X1-1.KL; no longer CASE1-3.KL, SJ4.2
- net D2: now also SL030.5; no longer JP1.7
- net D3: now also 5V_SSR_CON-1.KL, SJ4.2; no longer JP1.6
- net D4: now also 5V_SSR_CON-3.KL, SJ1.2; no longer JP1.5
- net D5: now also JP1.3; no longer CASE-1.KL
- net D6: now also JP1.1; no longer SL030.5
- net D7: now also JP1.2; no longer JP1.9
- net D8: now also JP1.4; no longer JP1.8
- net D9: now also JP1.6; no longer SG1.2
- net GND: now also 5V_SSR_CON-2.KL, 5V_SSR_CON-4.KL, X1-2.KL; no longer CASE-2.KL, CASE1-2.KL, CASE1-4.KL
- net N$25: now also RELAY1-1.KL; no longer RELAY-1.KL
- net N$27: now also RELAY1-2.KL; no longer RELAY-2.KL
- net N$29: now also RELAY1-3.KL; no longer RELAY-3.KL
- net N$30: now also RELAY1-4.KL; no longer RELAY-4.KL
- net N$31: now also RELAY1-5.KL; no longer RELAY-5.KL
- net N$32: now also RELAY1-6.KL; no longer RELAY-6.KL
- net N$42: now also RELAY2-4.KL; no longer RELAY1-1.KL
- net N$43: now also RELAY2-5.KL; no longer RELAY1-2.KL
- net N$46: now also RELAY2-2.KL; no longer RELAY1-5.KL
- net N$47: now also RELAY2-1.KL; no longer RELAY1-6.KL
- net RAW: now also POWER-2.KL; no longer POWER-6.KL
- net RESET: now also JP1.8; no longer JP1.4
- net VCC: now also POWER-6.KL; no longer POWER-4.KL, R13.2, R14.2
Other:
- moved on the sheet: RELAY1-1, RELAY1-2, RELAY1-3, RELAY1-4, RELAY1-5, RELAY1-6
